File: Raspi_Photometer_v2.brd (EAGLE design)
At the start: 167 x 94.9 mm, 52 parts, among them Q1 MMBT4403, Q2 32.768 KHz, T1 BC337, U1 HX711

Commit message: Add files via upload
Parts:
- removed T1: BC337, transistor:TO92
- added ADS115: (no value), con-amp-quick:10P
- added C14: 1uF, rcl (2):E2,5-5
- added C15: 220uF/50V, rcl:E5-10,5
- added IC1: (no value), SparkFun-PowerIC:SOT223
- added LCD_BACK: (no value), con-amp-quick:09P
- added R16: 3.3k, CEDTv83 (2):0207/7
- added R17, R18, R19: 100k, CEDTv83 (2):0207/7
- added R20: 100, CEDTv83 (2):0207/7
- CLKOUT1: value LED3MM -> LED1206; device CEDT_2016_V1:LED3MM -> CEDT_2016_V1:CHIPLED_1206
- Q1: device SparkFun-DiscreteSemi:SOT23-3 -> transistor-neu-to92:TO92-EBC
- R1, R2: device SparkFun-Resistors:0603-RES -> rcl:0204/7
- R10, R11, R7, R8, R9: value (none) -> 10k
- R12: value 20k -> 91K
- R13: value 3.3k -> 10K
- R14: value (none) -> 22k; device rcl:0204/7 -> CEDTv83 (2):0207/7
- U$1, U$2, U$3, U$4, U$5: value OMRON_SWITCH_10-XX -> OMRON_SWITCH_40-XX; device CEDT_JANUARY_2015_v5:B3F-10XX -> CEDT_JANUARY_2015_v5:B3F-40XX
- moved R14 78.3 mm to (-1.27, -6.35), turned to 0 degrees
- moved L1 17.7 mm to (52.1, 10.8), turned to 90 degrees
- moved C10 11.3 mm to (83.8, 11.4), turned to 270 degrees
- moved C12 5.99 mm to (78.1, 22.2)
- moved C11 2.01 mm to (69.8, 24.1)
- moved Q1 1.93 mm to (41.7, 53.6), flipped to the top, turned to 90 degrees
- moved C8 1.42 mm to (67.3, 23.5)
- renumbered TFT1 to LCD_FRONT
Connections:
- removed net 9V: C10.+, C12.+, D3.C, R12.2
- removed net EN: R14.2, T1.1, U$6.P$6
- new net +12V: C10.+, C12.+, D3.C, IC1.3, R12.2
- new net +9V: C15.+, IC1.2, R14.2, R18.2
- new net A2: ADS115.9
- new net A3: ADS115.10
- new net ALRT: ADS115.6
- new net N$18: C14.+, IC1.1, R14.1, R16.2
- new net N$20: R17.1, R18.1, R19.2
- new net P_VALUE: J1.P$2, R17.2
- new net SCL: ADS115.3
- new net SDA: ADS115.4
- net 3.3V: now also ADS115.1, LCD_BACK.1, Q1.E; no longer Q1.2
- net 5V: no longer T1.3
- net A+: now also ADS115.7, R19.1, R20.1; no longer J1.P$2
- net A-: no longer J2.P$2
- net E+: now also Q1.C; no longer Q1.3
- net GND: now also ADS115.2, ADS115.5, ADS115.8, C14.-, C15.-, J2.P$2, LCD_BACK.2, R16.1, R20.2; no longer R14.1
- net GPIO10: now also LCD_BACK.6
- net GPIO11: now also LCD_BACK.7
- net GPIO13: now also LCD_BACK.4
- net GPIO19: now also U$6.P$6; no longer T1.2
- net GPIO5: now also LCD_BACK.5
- net GPIO6: now also LCD_BACK.8
- net GPIO8: now also LCD_BACK.3
- net GPIO9: now also LCD_BACK.9
- net N$19: now also CLKOUT1.C; no longer CLKOUT1.K
- net N$4: now also Q1.B; no longer Q1.1
Routing:
- net A-: track 145.9 -> 0.00 mm
- net A+: track 122.8 -> 0.00 mm
- net GND: track 450.7 -> 401.0 mm
- net EN: track 40.5 -> 0.00 mm, vias 2 -> 0
- net 5V: track 107.0 -> 136.2 mm
- net 9V: track 21.2 -> 0.00 mm
- net E+: track 16.2 -> 3.10 mm
- net 3.3V: track 255.1 -> 245.0 mm
- net GPIO19: track 8.94 -> 0.18 mm
- net N$4: track 4.72 -> 0.09 mm
- net N$16: track 34.7 -> 38.7 mm
- net N$6: track 5.88 -> 2.91 mm
- net GPIO16: track 73.1 -> 75.9 mm
- net GPIO12: track 98.6 -> 101.3 mm
- net N$19: track 5.61 -> 7.54 mm
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
Commit message: Add files via upload
Parts:
- removed ADS115: (no value), con-amp-quick:10P
- added CON1: (no value), CEDT_July_2014:NEB21R
- added IC2: LM358MX, CEDT_July_2014:SO08
- added IC3, IC4: LM336LP, linear:TO92
- added JP1, JP2, JP3: (no value), jumper:SJ_2
- added R21: 10K, CEDTv83 (2):0207/7
- added R22: 1MEG, CEDTv83 (2):0207/7
- added R31, R32: 22K, CEDTv83 (2):0207/7
- added R41: 2K, CEDTv83 (2):0207/7
- added SL1: (no value), CEDT_JANUARY_2015_v5:02P
- C13: device rcl:C025-024X044 -> rcl:C0805
- R17: value 100k -> 68K
- R18: value 100k -> 2K
- R3: device SparkFun-Resistors:0603-RES -> rcl:0207/15
- R4, R5: device SparkFun-Resistors:0603-RES -> rcl:0207/7
- moved R20 161.2 mm to (127.9, 64.8), turned to 90 degrees
- moved R17 158.3 mm to (127.9, 74.9), turned to 90 degrees
- moved R19 156.2 mm to (125.3, 64.8), turned to 90 degrees
- moved R18 154.5 mm to (139.3, 42.5)
- moved LCD_BACK 139.5 mm to (108.2, 38.1), turned to 180 degrees
- moved Q1 123.6 mm to (163.1, 76.6), turned to 270 degrees
- moved C7 117.8 mm to (154.1, 72.6), turned to 0 degrees
- moved C3 116.5 mm to (155.2, 75.4), turned to 0 degrees
- moved R1 115.7 mm to (157.6, 76.8), turned to 270 degrees
- moved C14 115.3 mm to (101.2, 10.8), turned to 90 degrees
- moved R2 113.1 mm to (154.2, 82.7)
- moved C2 109.0 mm to (152.1, 69.6), turned to 0 degrees
- moved R3 105.4 mm to (147.8, 78.6), turned to 270 degrees
- moved C6 104.3 mm to (147.4, 81.7), turned to 90 degrees
- moved C1 103.8 mm to (149.6, 70.1), turned to 270 degrees
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Connections:
- removed net A-: R3.1
- removed net A2: ADS115.9
- removed net A3: ADS115.10
- removed net ALRT: ADS115.6
- removed net E+: C3.1, C7.1, Q1.C, R1.2, U1.3
- removed net SCL: ADS115.3
- removed net SDA: ADS115.4
- new net 5V_V2: IC2.1, IC2.2, R31.2
- new net A+1: JP1.1, R4.1
- new net A+2: JP1.3
- new net AVDD1: JP2.2, U1.3
- new net AVDD2: C3.1, C7.1, JP2.3, Q1.C, R1.2
- new net N$17: IC2.3, IC3.2, R41.2
- new net N$21: R18.2, R41.1
- new net N$22: IC3.3, IC4.2
- new net P_VALUE_V2: R17.2, R21.2, R22.1
- new net VFB1: JP3.2, U1.4
- new net VFB2: JP3.3, R1.1, R2.2
- net +9V: now also CON1.+, IC2.8, R18.1; no longer R18.2
- net 3.3V: now also JP2.1; no longer ADS115.1
- net A+: now also JP1.2, SL1.2; no longer ADS115.7, R4.1
- net GND: now also CON1.-, IC2.4, IC4.3, JP3.1, R22.2, R3.1, SL1.1; no longer ADS115.2, ADS115.5, ADS115.8
- net GPIO13: no longer LCD_BACK.4, LCD_FRONT.RST
- net GPIO15: now also U1.12
- net GPIO17: no longer U1.11
- net GPIO18: now also U1.11
- net GPIO22: now also LCD_BACK.4, LCD_FRONT.RST
- net GPIO27: no longer U1.12
- net N$20: now also R32.1; no longer R18.1
- net N$6: now also R31.1, R32.2; no longer R1.1, R2.2, U1.4
- net P_VALUE: now also R21.1; no longer R17.2
Routing:
- net GND: track 401.0 -> 724.4 mm
- net GPIO13: track 320.7 -> 0.00 mm, vias 2 -> 0
- net GPIO9: track 374.0 -> 112.0 mm, vias 2 -> 4
- net GPIO11: track 355.8 -> 111.5 mm, vias 0 -> 4
- net GPIO10: track 370.2 -> 127.6 mm, vias 0 -> 4
- net GPIO6: track 338.8 -> 96.6 mm, vias 0 -> 4
- net GPIO5: track 339.2 -> 114.9 mm, vias 2 -> 4
- net +9V: track 0.00 -> 210.4 mm, vias 0 -> 4
- net GPIO22: track 0.00 -> 162.6 mm, vias 0 -> 4
- net N$5: track 90.9 -> 195.9 mm, vias 0 -> 2
- net 3.3V: track 245.0 -> 332.5 mm
- net GPIO23: track 80.1 -> 5.23 mm
- net GPIO15: track 0.00 -> 67.5 mm
- net GPIO24: track 64.0 -> 131.2 mm, vias 0 -> 4
- net GPIO18: track 0.00 -> 67.0 mm
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Other:
- board size 167 x 94.9 mm -> 188.8 x 105.5 mm

Commit message: Add files via upload
Parts:
- C13: value (none) -> 0.1uF
Routing:
- net P_VALUE: track 9.26 -> 11.1 mm
- net GND: track 724.4 -> 723.0 mm
