File: Raspi_Photometer_v2.sch (EAGLE design)
At the start: 52 parts, among them Q1 MMBT4403, Q2 32.768 KHz, T1 BC337, U1 HX711

Commit message: Add files via upload
Parts:
- removed T1: BC337, transistor:BC337
- added ADS115: (no value), con-amp-quick:M10
- added C14: 1uF, rcl (2):CPOL-EUE2.5-5
- added C15: 220uF/50V, rcl:CPOL-EUE5-10.5
- added IC1: (no value), SparkFun-PowerIC:V_REG_LM1117SOT223
- added LCD_BACK: (no value), con-amp-quick:M09
- added R16: 3.3k, CEDTv83 (2):RESISTOR0207/7
- added R17, R18, R19: 100k, CEDTv83 (2):RESISTOR0207/7
- added R20: 100, CEDTv83 (2):RESISTOR0207/7
- CLKOUT1: value LED3MM -> LED1206; device CEDT_2016_V1:LED3MM -> CEDT_2016_V1:LED1206
- Q1: device SparkFun-DiscreteSemi:TRANSISTOR_PNPMMBT4403 -> transistor-neu-to92:2N4403-PNP-TO92-EBC
- R1: device SparkFun-Resistors:20KOHM1/10W1%(0603) -> rcl:R-US_0204/7
- R10, R11, R7, R8, R9: value (none) -> 10k
- R12: value 20k -> 91K
- R13: value 3.3k -> 10K
- R14: value (none) -> 22k; device rcl:R-US_0204/7 -> CEDTv83 (2):RESISTOR0207/7
- R2: device SparkFun-Resistors:8.2KOHM-1/10W-5%(0603) -> rcl:R-US_0204/7
- U$1, U$2, U$3, U$4, U$5: value OMRON_SWITCH_10-XX -> OMRON_SWITCH_40-XX; device CEDT_JANUARY_2015_v5:OMRON_SWITCH_10-XX -> CEDT_JANUARY_2015_v5:OMRON_SWITCH_40-XX
- renumbered TFT1 to LCD_FRONT
Connections:
- removed net 9V: C10.+, C12.+, D3.C, R12.2
- removed net EN: R14.2, T1.E, U$6.EN
- new net +12V: C10.+, C12.+, D3.C, IC1.IN, R12.2
- new net +9V: C15.+, IC1.OUT, R14.2, R18.2
- new net A2: ADS115.9
- new net A3: ADS115.10
- new net ALRT: ADS115.6
- new net N$18: C14.+, IC1.ADJ, R14.1, R16.2
- new net N$20: R17.1, R18.1, R19.2
- new net P_VALUE: J1.1, R17.2
- new net SCL: ADS115.3
- new net SDA: ADS115.4
- net 3.3V: now also ADS115.1, LCD_BACK.1
- net 5V: no longer T1.C
- net A+: now also ADS115.7, R19.1, R20.1; no longer J1.1
- net A-: no longer J2.1
- net GND: now also ADS115.2, ADS115.5, ADS115.8, C14.-, C15.-, J2.1, LCD_BACK.2, R16.1, R20.2; no longer R14.1
- net GPIO10: now also LCD_BACK.6
- net GPIO11: now also LCD_BACK.7
- net GPIO13: now also LCD_BACK.4
- net GPIO19: now also U$6.EN; no longer T1.B
- net GPIO5: now also LCD_BACK.5
- net GPIO6: now also LCD_BACK.8
- net GPIO8: now also LCD_BACK.3
- net GPIO9: now also LCD_BACK.9
Other:
- note added: "*Photometer 9V using DC Jack??"
- note added: "AVDD jumper to 3.3V"
- note added: "VFB Jumper to GND"
- note added: "replace pushbuttons with 40XX"
- moved on the sheet: C10, C11, C12, C8, D3, J1, J2, L1, R12, R13, R14

Commit message: Add files via upload
Parts:
- removed ADS115: (no value), con-amp-quick:M10
- added CON1: (no value), CEDT_July_2014:POWER_CON
- added IC2: LM358MX, CEDT_July_2014:LM358MX
- added IC3, IC4: LM336LP, linear:LM336LP
- added JP1, JP2, JP3: (no value), jumper:SJ2W
- added R21: 10K, CEDTv83 (2):RESISTOR0207/7
- added R22: 1MEG, CEDTv83 (2):RESISTOR0207/7
- added R31, R32: 22K, CEDTv83 (2):RESISTOR0207/7
- added R41: 2K, CEDTv83 (2):RESISTOR0207/7
- added SL1: (no value), CEDT_JANUARY_2015_v5:M02
- C13: device rcl:C-US025-024X044 -> rcl:C-USC0805
- R17: value 100k -> 68K
- R18: value 100k -> 2K
- R3: device SparkFun-Resistors:100OHM-1/10W-1%(0603) -> rcl:R-US_0207/15
- R4: device SparkFun-Resistors:100OHM-1/10W-1%(0603) -> rcl:R-US_0207/7
- R5: device SparkFun-Resistors:10KOHM-1/10W-1%(0603)0603 -> rcl:R-US_0207/7
Connections:
- removed net A-: R3.1
- removed net A2: ADS115.9
- removed net A3: ADS115.10
- removed net ALRT: ADS115.6
- removed net E+: C3.1, C7.1, Q1.C, R1.2, U1.AVDD
- removed net SCL: ADS115.3
- removed net SDA: ADS115.4
- new net 5V_V2: IC2A.-IN, IC2A.OUT, R31.2
- new net A+1: JP1.1, R4.1
- new net A+2: JP1.3
- new net AVDD1: JP2.2, U1.AVDD
- new net AVDD2: C3.1, C7.1, JP2.3, Q1.C, R1.2
- new net N$17: IC2A.+IN, IC3.C, R41.2
- new net N$21: R18.2, R41.1
- new net N$22: IC3.A, IC4.C
- new net P_VALUE_V2: R17.2, R21.2, R22.1
- new net VFB1: JP3.2, U1.VFB
- new net VFB2: JP3.3, R1.1, R2.2
- net +9V: now also CON1.+, IC2P.V+, R18.1; no longer R18.2
- net 3.3V: now also JP2.1; no longer ADS115.1
- net A+: now also JP1.2, SL1.2; no longer ADS115.7, R4.1
- net GND: now also CON1.-, IC2P.V-, IC4.A, JP3.1, R22.2, R3.1, SL1.1; no longer ADS115.2, ADS115.5, ADS115.8
- net GPIO13: no longer LCD_BACK.4, LCD_FRONT.RST
- net GPIO15: now also U1.DOUT
- net GPIO17: no longer U1.PD_SCK
- net GPIO18: now also U1.PD_SCK
- net GPIO22: now also LCD_BACK.4, LCD_FRONT.RST
- net GPIO27: no longer U1.DOUT
- net N$20: now also R32.1; no longer R18.1
- net N$6: now also R31.1, R32.2; no longer R1.1, R2.2, U1.VFB
- net P_VALUE: now also R21.1; no longer R17.2
Other:
- note removed: "*Photometer 9V using DC Jack??"
- note removed: "AVDD jumper to 3.3V"
- note removed: "VFB Jumper to GND"
- moved on the sheet: J1, J2, R17, R18, R19, R20

Commit message: Add files via upload
Parts:
- C13: value (none) -> 0.1uF
Changed lines of the file:
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@@
 <part name="GND12" library="01_FAB_Hello (2)" deviceset="GND" device=""/>
 <part name="LCD_FRONT" library="CEDT_JANUARY_2015_v4" deviceset="TFT_LCD_2.2" device=""/>
-<part name="C13" library="rcl" deviceset="C-US" device="C0805"/>
+<part name="C13" library="rcl" deviceset="C-US" device="C0805" value="0.1uF"/>
 <part name="CLKOUT1" library="CEDT_2016_V1" deviceset="LED" device="1206" value="LED1206"/>
 <part name="R15" library="rcl" deviceset="R-US_" device="0204/7" value="330"/>
